File: Schmatic/PruebaDeEsquema/PruebaDeEsquema.kicad_sch (KiCad schematic)
At the start: 48 parts, among them J2 Conn_01x02_Pin, U3 TLV1117-33, U4 TLV4888, U5 TLV4888, U6 TLV1117-ADJ

Commit message: Improve ECG filter and supply robustness
Parts:
- added C15, C17: 100n, Capacitor_SMD:C_0805_2012Metric_Pad1.18x1.45mm_HandSolder, symbol Device:C
- added C16, C18: 10uF, Capacitor_SMD:C_0805_2012Metric_Pad1.18x1.45mm_HandSolder, symbol Device:C_Polarized_US
- added R39, R40, R41: 100R, Resistor_SMD:R_0805_2012Metric_Pad1.20x1.40mm_HandSolder, symbol Device:R
Connections:
- net -BATT_REG: now also C18.2
- net GND: now also C16.2, C18.1
- net HPF_out: now also R39.2; no longer R14.2, R17.2, U5.1
- net LPF_out: now also R41.2; no longer C11.2, R21.2, U5.8
- net N50Hz_out: now also R40.2; no longer C5.1, C8.1, R10.2, U5.7
- new net: C11.2, R21.2, R41.1, U5.8
- new net: C5.1, C8.1, R10.2, R40.1, U5.7
- new net: R14.2, R17.2, R39.1, U5.1
- new net +BATT_REG: C16.1
Other:
- note added: "| Robustez de filtrado y alimentacion | C15/C17: 100 nF ceramicos pegados a U4/U5. C16/C18: reserva local de 10 uF por riel. Mantener retornos cortos a GND para que el filtrado no module la alimentacion. | Propuestas de IC/activos | 1) Cambiar TLV4888 por OPAx333 / OPA4340 si se requiere menor offset y deriva. 2) Considerar AD8232/AD8233 como front-end ECG dedicado con right-leg-drive. 3) Usar re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"
